Commit message: Testes de simulacao com multi-robos, tentando resolver o uso de controladores individuais para cada robo

File: description/robot.urdf_2.xacro (robot description, xacro)
@@ -1,6 +1,9 @@
 <?xml version="1.0"?>
-<robot name="prm_robot"
-  xmlns:xacro="http://ros.org/wiki/xacro">
-  <!-- Definicao de Algumas Contantes -->
+<robot xmlns:xacro="http://www.ros.org/wiki/xacro" name="$(arg robot_name)">
+  <!-- Definicao do argumento nome do robo -->
+  <xacro:arg name="robot_name" default="prm_robot"/>
+  <!-- Definicao de propriedade com nome do robo -->
+  <xacro:property name="robot_name" value="$(arg robot_name)"/>
+  <xacro:property name="name_prefix" value="${robot_name}"/>
   <xacro:property name="base_width" value="0.31"/> <!-- Largura da base -->
   <xacro:property name="base_length" value="0.42"/> <!-- Comprimento da base -->
@@ -33,5 +36,5 @@
     </inertial>
   </xacro:macro>
-  <!-- Definindo plugin para publiar a pose do robo -->
+  <!-- Definindo plugin para publiar a pose do robo (posição geral de todo modelo)-->
   <gazebo>
     <plugin filename="libignition-gazebo-pose-publisher-system" name="ignition::gazebo::systems::PosePublisher">
@@ -45,5 +48,5 @@
   </gazebo>
   <!-- Definindo a Base do Robô -->
-  <link name="base_link">
+  <link name="${name_prefix}_base_link">
     <visual>
       <geometry>
@@ -62,10 +65,10 @@
   </link>
   <!-- Definindo a Base do Robô (base footprint) -->
-  <link name="base_footprint">
+  <link name="${name_prefix}_base_footprint">
     <xacro:box_inertia m="0" w="0" d="0" h="0"/>
   </link>
-  <joint name="base_joint" type="fixed">
-    <parent link="base_link"/>
-    <child link="base_footprint"/>
+  <joint name="${name_prefix}_base_joint" type="fixed">
+    <parent link="${name_prefix}_base_link"/>
+    <child link="${name_prefix}_base_footprint"/>
     <origin xyz="0.0 0.0 ${-(wheel_radius+wheel_zoff)}" rpy="0 0 0"/>
   </joint>
@@ -73,5 +76,5 @@
   <!-- Parâmetros: prefix: drivewhl_l, drivewhl_r -->
   <xacro:macro name="wheel" params="prefix x_reflect y_reflect">
-    <link name="${prefix}_link">
+    <link name="${name_prefix}_${prefix}_link">
       <visual>
         <origin xyz="0 0 0" rpy="${pi/2} 0 0"/>
@@ -91,7 +94,7 @@
       <xacro:cylinder_inertia m="2.5" r="${wheel_radius}" h="${wheel_width}"/>
     </link>
-    <joint name="${prefix}_joint" type="continuous">
-      <parent link="base_link"/>
-      <child link="${prefix}_link"/>
+    <joint name="${name_prefix}_${prefix}_joint" type="continuous">
+      <parent link="${name_prefix}_base_link"/>
+      <child link="${name_prefix}_${prefix}_link"/>
       <origin xyz="${x_reflect*wheel_xoff} ${y_reflect*(base_width/2+wheel_ygap)} ${-wheel_zoff}" rpy="0 0 0"/>
       <axis xyz="0 1 0"/>
@@ -101,5 +104,5 @@
   <xacro:wheel prefix="drivewhl_l" x_reflect="-1" y_reflect="1" />
   <xacro:wheel prefix="drivewhl_r" x_reflect="-1" y_reflect="-1" />
-  <link name="front_caster">
+  <link name="${name_prefix}_front_caster">
     <visual>
       <geometry>
@@ -118,11 +121,11 @@
     <xacro:sphere_inertia m="0.005" r="${(wheel_radius+wheel_zoff-(base_height/2))}"/>
   </link>
-  <joint name="caster_joint" type="fixed">
-    <parent link="base_link"/>
-    <child link="front_caster"/>
+  <joint name="${name_prefix}_caster_joint" type="fixed">
+    <parent link="${name_prefix}_base_link"/>
+    <child link="${name_prefix}_front_caster"/>
     <origin xyz="${caster_xoff} 0.0 ${-(base_height/2)}" rpy="0 0 0"/>
   </joint>
   <!-- Definindo a IMU do Robô (física) -->
-  <link name="imu_link">
+  <link name="${name_prefix}_imu_link">
     <visual>
       <geometry>
@@ -138,10 +141,10 @@
   </link>
   <!-- Definindo o sensor IMU no Gazebo -->
-  <gazebo reference="imu_link">
-    <sensor name="imu_sensor" type="imu">
-      <ignition_frame_id>imu_link</ignition_frame_id>
+  <gazebo reference="${name_prefix}_imu_link">
+    <sensor name="${name_prefix}_imu_sensor" type="imu">
+      <ignition_frame_id>${name_prefix}_imu_link</ignition_frame_id>
       <plugin filename="ignition-gazebo-imu-system" name="ignition::gazebo::systems::Imu">
       </plugin>
-      <topic>imu</topic>
+      <topic>${robot_name}/imu</topic>
       <always_on>true</always_on>
       <update_rate>50</update_rate>
@@ -204,61 +207,51 @@
   </gazebo>
   <!-- Ligando a IMU a base do robô -->
-  <joint name="imu_joint" type="fixed">
-    <parent link="base_link"/>
-    <child link="imu_link"/>
+  <joint name="${name_prefix}_imu_joint" type="fixed">
+    <parent link="${name_prefix}_base_link"/>
+    <child link="${name_prefix}_imu_link"/>
     <origin xyz="0 0 0.01"/>
   </joint>
-<!-- Define um sistema de controle ROS 2 utilizando a infraestrutura ros2_control -->
-<ros2_control name="IgnitionSystem" type="system">
-  <!-- Seção de hardware do sistema, onde é especificado o plugin que fará a ponte entre o Gazebo (Ignition) e o ros2_control -->
-  <hardware>
-    <!-- Plugin que permite a integração entre o Ignition Gazebo e o framework ros2_control -->
-    <plugin>ign_ros2_control/IgnitionSystem</plugin>
-  </hardware>
-  <!-- Definição do primeiro atuador, correspondente à roda esquerda ("drive wheel left") -->
-  <joint name="drivewhl_l_joint">
-    <!-- Interface de comando de velocidade angular (por exemplo, rad/s) para essa junta -->
-    <command_interface name="velocity">
-      <!-- Valor mínimo permitido para o comando de velocidade (limite inferior) -->
-      <param name="min">-1</param>
-      <!-- Valor máximo permitido para o comando de velocidade (limite superior) -->
-      <param name="max">1</param>
-    </command_interface>
-    <!-- Interface de estado que fornece a posição atual da junta (por exemplo, em radianos) -->
-    <state_interface name="position"/>
-    <!-- Interface de estado que fornece a velocidade atual da junta (por exemplo, em rad/s) -->
-    <state_interface name="velocity"/>
-  </joint>
-  <!-- Definição do segundo atuador, correspondente à roda direita ("drive wheel right") -->
-  <joint name="drivewhl_r_joint">
-    <!-- Interface de comando de velocidade angular para essa junta -->
-    <command_interface name="velocity">
-      <!-- Limite inferior da velocidade que pode ser comandada -->
-      <param name="min">-1</param>
-      <!-- Limite superior da velocidade que pode ser comandada -->
-      <param name="max">1</param>
-    </command_interface>
-    <!-- Interface de estado para leitura da posição da junta -->
-    <state_interface name="position"/>
-    <!-- Interface de estado para leitura da velocidade da junta -->
-    <state_interface name="velocity"/>
-  </joint>
-</ros2_control>
-  <gazebo>
+  <!-- Define um sistema de controle ROS 2 utilizando a infraestrutura ros2_control -->
+  <ros2_control name="IgnitionSystem" type="system">
+    <!-- Seção de hardware do sistema, onde é especificado o plugin que fará a ponte entre o Gazebo (Ignition) e o ros2_control -->
+    <hardware>
+      <!-- Plugin que permite a integração entre o Ignition Gazebo e o framework ros2_control -->
+      <plugin>ign_ros2_control/IgnitionSystem</plugin>
+    </hardware>
+    <!-- Definição do primeiro atuador, correspondente à roda esquerda ("drive wheel left") -->
+    <joint name="${name_prefix}_drivewhl_l_joint">
+      <!-- Interface de comando de velocidade angular (por exemplo, rad/s) para essa junta -->
+      <command_interface name="velocity">
+        <!-- Valor mínimo permitido para o comando de velocidade (limite inferior) -->
+        <param name="min">-1</param>
+        <!-- Valor máximo permitido para o comando de velocidade (limite superior) -->
+        <param name="max">1</param>
+      </command_interface>
+      <!-- Interface de estado que fornece a posição atual da junta (por exemplo, em radianos) -->
+      <state_interface name="position"/>
+      <!-- Interface de estado que fornece a velocidade atual da junta (por exemplo, em rad/s) -->
+      <state_interface name="velocity"/>
+    </joint>
+    <!-- Definição do segundo atuador, correspondente à roda direita ("drive wheel right") -->
+    <joint name="${name_prefix}_drivewhl_r_joint">
+      <!-- Interface de comando de velocidade angular para essa junta -->
+      <command_interface name="velocity">
+        <!-- Limite inferior da velocidade que pode ser comandada -->
+        <param name="min">-1</param>
+        <!-- Limite superior da velocidade que pode ser comandada -->
+        <param name="max">1</param>
+      </command_interface>
+      <!-- Interface de estado para leitura da posição da junta -->
+      <state_interface name="position"/>
+      <!-- Interface de estado para leitura da velocidade da junta -->
+      <state_interface name="velocity"/>
+    </joint>
+  </ros2_control>
+  <gazebo reference="${name_prefix}_base_link">
     <plugin filename="ign_ros2_control-system" name="ign_ros2_control::IgnitionROS2ControlPlugin">
       <parameters>$(find prm)/config/diff_drive_controller_velocity.yaml</parameters>
     </plugin>
   </gazebo>
-  <!-- <gazebo> https://github.com/ros-controls/gz_ros2_control/issues/49
-    <plugin filename="ign_ros2_control-system" name="ign_ros2_control::IgnitionROS2ControlPlugin">
-      <controller_manager_prefix_node_name>prm_robot</controller_manager_prefix_node_name>
-      <parameters>$(find prm)/config/diff_drive_controller_velocity.yaml</parameters>
-      <ros>
-        <namespace>prm_robot</namespace>
-        <remapping>/tf:=/$(arg namespace)/tf</remapping>
-      </ros>
-    </plugin>
-  </gazebo> -->
-  <link name="lidar_link">
+  <link name="${name_prefix}_lidar_link">
     <inertial>
       <origin xyz="0 0 0" rpy="0 0 0"/>
@@ -282,13 +275,13 @@
     </visual>
   </link>
-  <joint name="lidar_joint" type="fixed">
-    <parent link="base_link"/>
-    <child link="lidar_link"/>
+  <joint name="${name_prefix}_lidar_joint" type="fixed">
+    <parent link="${name_prefix}_base_link"/>
+    <child link="${name_prefix}_lidar_link"/>
     <origin xyz="0 0 0.12" rpy="0 0 0"/>
   </joint>
-  <gazebo reference="lidar_link">
-    <sensor name="lidar" type="gpu_lidar">
-      <ignition_frame_id>lidar_link</ignition_frame_id>
-      <topic>scan</topic>
+  <gazebo reference="${name_prefix}_lidar_link">
+    <sensor name="${name_prefix}_lidar" type="gpu_lidar">
+      <ignition_frame_id>${name_prefix}_lidar_link</ignition_frame_id>
+      <topic>${robot_name}/scan</topic>
       <always_on>true</always_on>
       <visualize>true</visualize>
@@ -316,5 +309,5 @@
     </sensor>
   </gazebo>
-  <link name="camera_link">
+  <link name="${name_prefix}_camera_link">
     <visual>
       <origin xyz="0 0 0" rpy="0 0 0"/>
@@ -338,18 +331,18 @@
     </inertial>
   </link>
-  <joint name="camera_joint" type="fixed">
-    <parent link="base_link"/>
-    <child link="camera_link"/>
+  <joint name="${name_prefix}_camera_joint" type="fixed">
+    <parent link="${name_prefix}_base_link"/>
+    <child link="${name_prefix}_camera_link"/>
     <origin xyz="0.215 0 0.05" rpy="0 0 0"/>
   </joint>
-  <link name="camera_frame"/>
-  <joint name="camera_frame_joint" type="fixed">
+  <link name="${name_prefix}_camera_frame"/>
+  <joint name="${name_prefix}_camera_frame_joint" type="fixed">
     <origin xyz="0 0 0" rpy="${-pi/2} 0 ${-pi/2}"/>
-    <parent link="camera_link"/>
-    <child link="camera_frame"/>
-  </joint>
-  <gazebo reference="camera_link">
+    <parent link="${name_prefix}_camera_link"/>
+    <child link="${name_prefix}_camera_frame"/>
+  </joint>
+  <gazebo reference="${name_prefix}_camera_link">
     <!-- Insere uma camera comum RGB -->
-    <!-- <sensor name="robot_cam" type="camera">
+    <!-- <sensor name="${name_prefix}_robot_cam" type="camera">
       <camera>
         <horizontal_fov>1.57</horizontal_fov>
@@ -366,10 +359,10 @@
       <update_rate>15</update_rate>
       <visualize>true</visualize>
-      <topic>robot_cam</topic>
+      <topic>${robot_name}/robot_cam</topic>
       <enable_metrics>true</enable_metrics>
     </sensor> -->
     <!-- Insere uma camera com segmentacao semantica -->
-    <sensor name="robot_cam" type="segmentation">
-      <topic>robot_cam</topic>
+    <sensor name="${name_prefix}_robot_cam" type="segmentation">
+      <topic>${robot_name}/robot_cam</topic>
       <camera>
         <segmentation_type>semantic</segmentation_type>
@@ -389,6 +382,6 @@
     </sensor>
     <!-- Insere uma camera bounding box 2D completo -->
-    <!-- <sensor name="full_2d" type="boundingbox_camera">
-      <topic>boxes_full_2d</topic>
+    <!-- <sensor name="${name_prefix}_full_2d" type="boundingbox_camera">
+      <topic>${robot_name}/boxes_full_2d</topic>
       <camera>
         <box_type>full_2d</box_type>
@@ -411,6 +404,6 @@
     </sensor> -->
     <!-- Insere uma camera bounding box 2D -->
-    <!-- <sensor name="visible_2d" type="boundingbox_camera">
-      <topic>boxes_visible_2d</topic>
+    <!-- <sensor name="${name_prefix}_visible_2d" type="boundingbox_camera">
+      <topic>${robot_name}/boxes_visible_2d</topic>
       <camera>
         <box_type>visible_2d</box_type>
@@ -433,6 +426,6 @@
     </sensor> -->
     <!-- Insere uma camera bounding box 3D -->
-    <!-- <sensor name="3d" type="boundingbox_camera">
-      <topic>boxes_3d</topic>
+    <!-- <sensor name="${name_prefix}_3d" type="boundingbox_camera">
+      <topic>${robot_name}/boxes_3d</topic>
       <camera>
         <box_type>3d</box_type>
